Commit message: bug fixes and simulation file name changed

File: src/disaster_robot/urdf/disaster_robot.urdf.xacro (robot description, xacro)
@@ -65,9 +65,9 @@
   <link name="base_link">
     <visual>
-      <origin xyz="-0.064 0 0.0" rpy="0 0 0"/>
+      <origin xyz="-0.064 0 ${base_height/2}" rpy="0 0 0"/>
       <geometry>
         <box size="${base_length} ${base_width} ${base_height}"/>
       </geometry>
-      <material name="dark"/>
+      <material name="blue"/>
     </visual>
     <collision>
@@ -86,5 +86,5 @@
           <cylinder radius="${wheel_radius}" length="${wheel_width}"/>
         </geometry>
-        <material name="dark"/>
+        <material name="orange"/>
       </visual>
       <collision>
@@ -186,11 +186,11 @@
   </joint>
   <gazebo reference="base_link">
-    <material>Gazebo/DarkGrey</material>
+    <material>Gazebo/Blue</material>
   </gazebo>
   <gazebo reference="left_wheel_link">
-    <material>Gazebo/FlatBlack</material>
+    <material>Gazebo/Orange</material>
   </gazebo>
   <gazebo reference="right_wheel_link">
-    <material>Gazebo/FlatBlack</material>
+    <material>Gazebo/Orange</material>
   </gazebo>
   <gazebo reference="camera_link">
@@ -216,5 +216,5 @@
       <robot_base_frame>base_footprint</robot_base_frame>
       <publish_odom>true</publish_odom>
-      <publish_odom_tf>false</publish_odom_tf>
+      <publish_odom_tf>true</publish_odom_tf>
       <max_wheel_torque>20</max_wheel_torque>
       <max_wheel_acceleration>1.0</max_wheel_acceleration>
